Commit message: Update

File: urdf/robot.urdf.xacro (robot description, xacro)
@@ -45,5 +45,5 @@
 		<collision name="collision_chassis">
 			<geometry>
-				<box size="${l1} ${b1} ${h1}"/>
+				<box size="${l1} ${b1} ${h1+b2+h1}"/>
 			</geometry>
 		</collision>
@@ -67,5 +67,5 @@
 		</visual>
 		<collision name="collision_right_wheel">
-		<origin rpy="0 1.5707 1.5707" xyz="0 0 0"/>
+			<origin rpy="0 1.5707 0" xyz="0 0 0"/>
 			<geometry>
 				<cylinder length="${l3}" radius="${r3}"/>
@@ -74,5 +74,5 @@
 		<inertial>
 			<mass value="0.2"/>
-			<origin rpy="0 1.5707 1.5707" xyz="0 0 0"/>
+				<origin rpy="0 1.5707 0" xyz="0 0 0"/>
 			<inertia ixx="${m3*((3*r3*r3)+(l3*l3))/12.0}" ixy="0" ixz="0" iyy="${m3*((3*r3*r3)+(l3*l3))/12.0}" iyz="0" izz="${(m3*r3*r3)/2.0}"/>
 		</inertial>
@@ -95,5 +95,5 @@
 		</visual>
 		<collision name="collision_left_wheel">
-		<origin rpy="0 1.5707 1.5707" xyz="0 0 0"/>
+			<origin rpy="0 1.5707 0" xyz="0 0 0"/>
 			<geometry>
 				<cylinder length="${l3}" radius="${r3}"/>
@@ -102,5 +102,5 @@
 		<inertial>
 			<mass value="0.2"/>
-			<origin rpy="0 1.5707 1.5707" xyz="0 0 0"/>
+			<origin rpy="0 1.5707 0" xyz="0 0 0"/>
 			<inertia ixx="${m3*((3*r3*r3)+(l3*l3))/12.0}" ixy="0" ixz="0" iyy="${m3*((3*r3*r3)+(l3*l3))/12.0}" iyz="0" izz="${(m3*r3*r3)/2.0}"/>
 		</inertial>
